Commit message: Refactor code structure for improved readability and maintainability

File: task_board.urdf.xacro (robot description, xacro)
@@ -3,4 +3,5 @@
   <xacro:arg name="load_round_belt_pulleys" default="false" />
   <xacro:arg name="load_timing_belt_pulleys" default="false" />
+  <xacro:arg name="load_bike_chain_pulleys" default="false" />
   <!-- board side length is .384m -->
   <link name="board">
@@ -21,4 +22,144 @@
     </collision>
   </link>
+  <!-- Bike Chain Pulleys -->
+  <xacro:if value="$(arg load_bike_chain_pulleys)">
+    <joint name="chain_tensioner_bracket_joint" type="fixed">
+      <parent link="board" />
+      <child link="chain_tensioner_bracket" />
+      <!-- <origin xyz="0.2395 0.347 0.020425" rpy="0 0 ${pi/2}" /> -->
+      <!-- .065 .0325-->
+      <!-- .311427 -->
+      <origin xyz="0.2395 0.343927 0.006" rpy="0 0 ${pi/2}" />
+      <axis xyz="1 0 0" />
+      <limit lower="-1.0" upper="1.0" effort="100" velocity="100" />
+    </joint>
+    <link name="chain_tensioner_bracket">
+      <visual>
+        <origin xyz="0 0 0" rpy="0 0 0" />
+        <geometry>
+          <mesh filename="bike_chain_task/tensioner_bracket.gltf" />
+        </geometry>
+      </visual>
+      <collision>
+        <origin xyz="0 0 0" rpy="0 0 0" />
+        <geometry>
+          <mesh filename="bike_chain_task/tensioner_bracket.gltf" />
+        </geometry>
+      </collision>
+      <inertial>
+        <mass value="1.0" />
+        <origin xyz="0 0 0" />
+        <inertia ixx="1.0" ixy="0.0" ixz="0.0" iyy="1.0" iyz="0.0" izz="1.0" />
+      </inertial>
+    </link>
+    <joint name="chain_tensioner_slide_joint" type="fixed">
+      <parent link="chain_tensioner_bracket" />
+      <child link="chain_tensioner_slide" />
+      <origin xyz="-0.021 0 0" rpy="0 0 0" />
+      <axis xyz="1 0 0" />
+      <limit lower="-1.0" upper="1.0" effort="100" velocity="100" />
+    </joint>
+    <!-- dummy link -->
+    <link name="chain_tensioner_slide">
+    </link>
+    <joint name="chain_tensioner_joint" type="prismatic">
+    <!-- .062 slide limit -->
+      <parent link="chain_tensioner_slide" />
+      <child link="chain_tensioner_sprocket" />
+      <origin xyz="0 0 0" rpy="0 0 0" />
+      <axis xyz="1 0 0" />
+      <limit lower="0" upper="0.04" effort="100" velocity="100" />
+    </joint>
+    <link name="chain_tensioner_sprocket">
+      <visual>
+        <origin xyz="0 0 0" rpy="${pi/2} 0 0" />
+        <geometry>
+          <mesh filename="bike_chain_task/tensioner_bolt.gltf" />
+        </geometry>
+        <material name="material_name">
+          <color rgba="1 1 1 1" />
+        </material>
+      </visual>
+      <visual>
+        <origin xyz="0 0 .015" rpy="0 ${-pi/2} 0" />
+        <geometry>
+          <mesh filename="bike_chain_task/tensioner_bearing.gltf" />
+        </geometry>
+        <material name="material_name">
+          <color rgba="1 1 1 1" />
+        </material>
+      </visual>
+      <visual>
+        <origin xyz="0 0 0.012" rpy="0 0 0" />
+        <geometry>
+          <mesh filename="bike_chain_task/tensioner_sprocket.obj" />
+        </geometry>
+        <material name="material_name">
+          <color rgba="1 1 1 1" />
+        </material>
+      </visual>
+      <collision>
+        <origin xyz="0 0 0" rpy="${pi/2} 0 0" />
+        <geometry>
+          <mesh filename="bike_chain_task/tensioner_bolt.gltf" />
+        </geometry>
+      </collision>
+      <inertial>
+        <mass value="1.0" />
+        <origin xyz="0 0 0" />
+        <inertia ixx="1.0" ixy="0.0" ixz="0.0" iyy="1.0" iyz="0.0" izz="1.0" />
+      </inertial>
+    </link>
+    <joint name="chain_small_sprocket_joint" type="fixed">
+      <parent link="board" />
+      <child link="chain_small_sprocket" />
+      <!-- <origin xyz="0.054 0.073 0.020" rpy="0 0 0" /> -->
+      <origin xyz="0.33 0.311 0.020" rpy="0 0 0" />
+    </joint>
+    <link name="chain_small_sprocket">
+      <visual>
+        <origin xyz="0 0 0" rpy="0 0 0" />
+        <geometry>
+          <mesh filename="bike_chain_task/small_sprocket.obj" />
+        </geometry>
+      </visual>
+      <collision>
+        <origin xyz="0 0 0" rpy="0 0 0" />
+        <geometry>
+          <mesh filename="bike_chain_task/small_sprocket.obj" />
+        </geometry>
+      </collision>
+      <inertial>
+        <mass value="1.0" />
+        <origin xyz="0 0 0" />
+        <inertia ixx="1.0" ixy="0.0" ixz="0.0" iyy="1.0" iyz="0.0" izz="1.0" />
+      </inertial>
+    </link>
+    <joint name="chain_large_sprocket_joint" type="fixed">
+      <parent link="board" />
+      <child link="chain_large_sprocket" />
+      <!-- <origin xyz="0.384 - 0.234 0.073 0.023" rpy="0 0 0" /> -->
+      <origin xyz="0.15 0.311 0.023" rpy="0 0 0" />
+    </joint>
+    <link name="chain_large_sprocket">
+      <visual>
+        <origin xyz="0 0 0" rpy="0 0 0" />
+        <geometry>
+          <mesh filename="bike_chain_task/large_sprocket.obj" />
+        </geometry>
+      </visual>
+      <collision>
+        <origin xyz="0 0 0" rpy="0 0 0" />
+        <geometry>
+          <mesh filename="bike_chain_task/large_sprocket.obj" />
+        </geometry>
+      </collision>
+      <inertial>
+        <mass value="1.0" />
+        <origin xyz="0 0 0" />
+        <inertia ixx="1.0" ixy="0.0" ixz="0.0" iyy="1.0" iyz="0.0" izz="1.0" />
+      </inertial>
+    </link>
+  </xacro:if>
   <!-- Round Belt Pulleys -->
   <xacro:if value="$(arg load_round_belt_pulleys)">

Commit message: Add timing belt tensioner components to task board URDF

File: task_board.urdf.xacro (robot description, xacro)
@@ -427,4 +427,77 @@
       <origin xyz="0 0 0" rpy="0 0 0"/>
     </joint>
+    <joint name="timing_belt_tensioner_joint" type="fixed">
+      <parent link="board" />
+      <child link="timing_belt_tensioner" />
+      <origin xyz="0.315 0.112 0" rpy="0 0 ${33*pi/50}" />
+      <axis xyz="1 0 0" />
+      <limit lower="-1.0" upper="1.0" effort="100" velocity="100" />
+    </joint>
+    <link name="timing_belt_tensioner">
+      <visual>
+        <origin xyz="0 0 0" rpy="0 0 0" />
+        <geometry>
+          <mesh filename="timing_belt_task/tensioner_base.gltf" />
+        </geometry>
+        <material name="material_name">
+          <color rgba="1 1 1 1" />
+        </material>
+      </visual>
+      <collision>
+        <origin xyz="0 0 0" rpy="0 0 0" />
+        <geometry>
+          <mesh filename="timing_belt_task/tensioner_base.gltf" />
+        </geometry>
+      </collision>
+      <inertial>
+        <mass value="1.0" />
+        <origin xyz="0 0 0" />
+        <inertia ixx="1.0" ixy="0.0" ixz="0.0" iyy="1.0" iyz="0.0" izz="1.0" />
+      </inertial>
+    </link>
+    <joint name="timing_belt_tensioner_arm_joint" type="revolute">
+      <parent link="timing_belt_tensioner" />
+      <child link="timing_belt_tensioner_arm" />
+      <origin xyz="0 0 0" rpy="0 0 0" />
+      <axis xyz="1 0 0" />
+      <limit lower="-1.0" upper="1.0" effort="100" velocity="100" />
+    </joint>
+    <link name="timing_belt_tensioner_arm">
+      <visual>
+        <origin xyz="0 0 0" rpy="0 0 0" />
+        <geometry>
+          <mesh filename="timing_belt_task/tensioner_arm.gltf" />
+        </geometry>
+        <material name="material_name">
+          <color rgba="1 1 1 1" />
+        </material>
+      </visual>
+      <visual>
+        <origin xyz="0 0.08 0.04492" rpy="${-pi/2} 0 0" />
+        <geometry>
+          <mesh filename="timing_belt_task/tensioner_rotary.gltf" />
+        </geometry>
+        <material name="material_name">
+          <color rgba="1 1 1 1" />
+        </material>
+      </visual>
+      <collision>
+        <origin xyz="0 0 0" rpy="0 0 0" />
+        <geometry>
+          <mesh filename="timing_belt_task/tensioner_arm.gltf" />
+        </geometry>
+      </collision>
+      <collision>
+        <origin xyz="0 0.08 0.04492" rpy="${-pi/2} 0 0" />
+        <geometry>
+          <mesh filename="timing_belt_task/tensioner_rotary.gltf" />
+        </geometry>
+      </collision>
+      <inertial>
+        <mass value="1.0" />
+        <origin xyz="0 0 0" />
+        <inertia ixx="1.0" ixy="0.0" ixz="0.0" iyy="1.0" iyz="0.0" izz="1.0" />
+      </inertial>
+    </link>
   </xacro:if>
 </robot>

Commit message: Add collision geometries for bike chain tensioner components in URDF

File: task_board.urdf.xacro (robot description, xacro)
@@ -100,4 +100,22 @@
       </visual>
       <collision>
+        <origin xyz="0 0 0.012" rpy="0 0 0" />
+        <geometry>
+          <mesh filename="bike_chain_task/tensioner_sprocket.obj" />
+        </geometry>
+        <material name="material_name">
+          <color rgba="1 1 1 1" />
+        </material>
+      </collision>
+      <collision>
+        <origin xyz="0 0 .015" rpy="0 ${-pi/2} 0" />
+        <geometry>
+          <mesh filename="bike_chain_task/tensioner_bearing.gltf" />
+        </geometry>
+        <material name="material_name">
+          <color rgba="1 1 1 1" />
+        </material>
+      </collision>
+      <collision>
         <origin xyz="0 0 0" rpy="${pi/2} 0 0" />
         <geometry>
