Commit message: Add collision geometries for table, wooden plate, base plate, and metal bar in URDF

File: common/scene.urdf.xacro (robot description, xacro)
@@ -3,12 +3,25 @@
     <!-- Root frame preserving the old top-level scene frame -->
     <link name="scene"/>
+    <!-- define constants -->
+    <!-- table OBB extents: array([1524.  ,  914.4 ,   44.45]) -->
+    <xacro:property name="table_height" value="0.04445"/>
+    <xacro:property name="table_length" value="1.524"/>
+    <xacro:property name="table_width" value="0.9144"/>
+    <xacro:property name="table_origin_z_offset" value="0.00255"/>
     <!-- Table -->
     <link name="table">
         <visual>
-            <origin rpy="0 0 0" xyz="0 0 0"/>
+            <!-- table mesh origin is 2.55mm floating above the table surface -->
+            <origin rpy="0 0 0" xyz="0 0 ${table_origin_z_offset}"/>
             <geometry>
                 <mesh filename="table/table.gltf" scale="0.001 0.001 0.001"/>
             </geometry>
         </visual>
+        <collision>
+            <origin rpy="0 0 0" xyz="0 0 ${-table_height/2}"/>
+            <geometry>
+                <box size="${table_length} ${table_width} ${table_height}"/>
+            </geometry>
+        </collision>
     </link>
     <joint name="scene_to_table" type="fixed">
@@ -17,4 +30,8 @@
         <origin rpy="0 0 ${pi/2}" xyz="0.23008 0 -0.02858"/>
     </joint>
+    <!-- Wooden board OBB extents: [914.4  304.8   19.05] -->
+    <xacro:property name="wooden_plate_length" value="0.9144"/>
+    <xacro:property name="wooden_plate_width" value="0.3048"/>
+    <xacro:property name="wooden_plate_height" value="0.01905"/>
     <!-- in x, table edge to wooden plate edge is 0.303 on one side and .306 on the other -->
     <!-- in y table edge to wooden plate edge is 0.3025 on one side and .3065 on the other -->
@@ -27,4 +44,11 @@
             </geometry>
         </visual>
+        <collision>
+            <origin rpy="0 0 0" xyz="0 0 ${-wooden_plate_height/2}"/>
+            <geometry>
+                <!-- array([914.4, 304.8, 19.05]) -->
+                <box size="${wooden_plate_length} ${wooden_plate_width} ${wooden_plate_height}"/>
+            </geometry>
+        </collision>
     </link>
     <joint name="table_to_wooden_plate" type="fixed">
@@ -33,4 +57,9 @@
         <origin rpy="0 0 0" xyz="0 0.30677 0.01905"/>
     </joint>
+    <!-- Base plate OBB extents: [0.254    0.254    0.009525] -->
+    <xacro:property name="base_plate_length" value="0.254"/>
+    <xacro:property name="base_plate_width" value="0.254"/>
+    <xacro:property name="base_plate_height" value="0.009525"/>
+    <xacro:property name="base_plate_to_franka_x_offset" value="0.0763"/>
     <!-- Base plate -->
     <link name="base_plate">
@@ -41,4 +70,11 @@
             </geometry>
         </visual>
+        <collision>
+            <origin rpy="0 0 0" xyz="0 ${-base_plate_to_franka_x_offset} ${-base_plate_height/2}"/>
+            <geometry>
+                <!-- array([0.254, 0.254, 0.009525]) -->
+                <box size="${base_plate_length} ${base_plate_width} ${base_plate_height}"/>
+            </geometry>
+        </collision>
     </link>
     <joint name="wooden_plate_to_base_plate" type="fixed">
@@ -47,3 +83,27 @@
         <origin rpy="0 0 ${-pi}" xyz="0 -0.07669 0.00953"/>
     </joint>
+    <xacro:property name="metal_bar_length" value="0.735"/>
+    <xacro:property name="metal_bar_width" value="0.048"/>
+    <xacro:property name="metal_bar_height" value="0.01"/>
+    <!-- metal bar length is 73.5cm -->
+    <!-- extends about 4.8cm from table edge -->
+    <link name="metal_bar">
+        <visual>
+            <origin rpy="0 0 0" xyz="0 0 ${-metal_bar_height/2}"/>
+            <geometry>
+                <box size="${metal_bar_length} ${metal_bar_width} ${metal_bar_height}"/>
+            </geometry>
+        </visual>
+        <collision>
+            <origin rpy="0 0 0" xyz="0 0 ${-metal_bar_height/2}"/>
+            <geometry>
+                <box size="${metal_bar_length} ${metal_bar_width} ${metal_bar_height}"/>
+            </geometry>
+        </collision>
+    </link>
+    <joint name="table_to_metal_bar" type="fixed">
+        <parent link="table"/>
+        <child link="metal_bar"/>
+        <origin rpy="0 0 0" xyz="0 ${-table_width/2 + metal_bar_width/2} ${metal_bar_height}"/>
+    </joint>
 </robot>

Commit message: Fix metal bar height value in URDF to match specifications

File: common/scene.urdf.xacro (robot description, xacro)
@@ -85,5 +85,5 @@
     <xacro:property name="metal_bar_length" value="0.735"/>
     <xacro:property name="metal_bar_width" value="0.048"/>
-    <xacro:property name="metal_bar_height" value="0.01"/>
+    <xacro:property name="metal_bar_height" value="0.0034"/>
     <!-- metal bar length is 73.5cm -->
     <!-- extends about 4.8cm from table edge -->

Commit message: Add franka workspace visualization and task bounding box to URDF

File: common/scene.urdf.xacro (robot description, xacro)
@@ -78,4 +78,54 @@
         </collision>
     </link>
+    <joint name="base_plate_to_franka_workspace_viz" type="fixed">
+        <parent link="base_plate"/>
+        <child link="franka_workspace_viz"/>
+        <origin rpy="0 0 0" xyz="0 0 0"/>
+    </joint>
+    <xacro:property name="franka_max_reach" value="0.855"/>
+    <xacro:property name="franka_min_reach" value="0.2"/>
+    <link name="franka_workspace_viz">
+        <visual>
+            <origin rpy="0 0 0" xyz="0 0 0"/>
+            <!-- make a transparent visualization of the franka workspace -->
+            <material name="franka_workspace_material">
+                <color rgba="0.0 0.0 1.0 0.15"/>
+            </material>
+            <geometry>
+                <sphere radius="${franka_max_reach}"/>
+            </geometry>
+        </visual>
+        <visual>
+            <origin rpy="0 0 0" xyz="0 0 0"/>
+            <!-- make a transparent visualization of the franka workspace -->
+            <material name="franka_workspace_material">
+                <color rgba="1.0 0.0 0.0 0.15"/>
+            </material>
+            <geometry>
+                <sphere radius="${franka_min_reach}"/>
+            </geometry>
+        </visual>
+    </link>
+    <joint name="table_to_task_bbox" type="fixed">
+        <parent link="table"/>
+        <child link="task_bbox"/>
+        <origin rpy="0 0 0" xyz="0 0 0"/>
+    </joint>
+    <xacro:property name="task_bbox_length" value="0.75"/>
+    <xacro:property name="task_bbox_width" value="0.48"/>
+    <xacro:property name="task_bbox_height" value="0.5"/>
+    <xacro:property name="table_to_task_bbox_y_offset" value="0.21"/>
+    <link name="task_bbox">
+        <visual>
+            <origin rpy="0 0 0" xyz="0 ${-table_to_task_bbox_y_offset} ${task_bbox_height/2}"/>
+            <!-- make a transparent visualization of the task bbox -->
+            <material name="task_bbox_material">
+                <color rgba="1.0 1.0 0.0 0.15"/>
+            </material>
+            <geometry>
+                <box size="${task_bbox_length} ${task_bbox_width} ${task_bbox_height}"/>
+            </geometry>
+        </visual>
+    </link>
     <joint name="wooden_plate_to_base_plate" type="fixed">
         <parent link="wooden_plate"/>

Commit message: slightly decrease task bbox height

File: common/scene.urdf.xacro (robot description, xacro)
@@ -114,5 +114,5 @@
     <xacro:property name="task_bbox_length" value="0.75"/>
     <xacro:property name="task_bbox_width" value="0.48"/>
-    <xacro:property name="task_bbox_height" value="0.5"/>
+    <xacro:property name="task_bbox_height" value="0.4"/>
     <xacro:property name="table_to_task_bbox_y_offset" value="0.21"/>
     <link name="task_bbox">
